File: massue_bento_v2_power.sch (KiCad schematic (older format))
At the start: 0 parts

Commit message: Add: power management schematic section
Parts:
- added C? (x3): 220uF, 6.3V, symbol CAPAPOL
- added C?: 470pF, symbol C
- added P? (x2): CONN_1, symbol CONN_1
- added R?: 2k, symbol R
- added U?: TC1015-3.3, symbol TC1015
- added U?: MCP73832, symbol MCP73832
Connections:
- new net: C?.1, U?.4 (BYPASS)
- new net: R?.1, U?.5 (PROG)
- new net +3.3V: C?.1, U?.5 (VOUT)
- new net +5V_USB: C?.1, U?.4 (VDD)
- new net GND: C?.2, C?.2, C?.2, C?.2, P?.1, R?.2, U?.2 (GND), U?.2 (VSS)
- new net LIPO_CHRG_STAT: U?.1 (STAT)
- new net VBAT: C?.1, P?.1, U?.1 (VIN), U?.3 (VBAT), U?.3 (~SHDN)
Other:
- note added: "3.3V regulator for MCU and sensors"
- note added: "Battery +"
- note added: "Battery -"
- note added: "Li-Po batt. charger from USB +5V input"
