File: massue_bento_v2.kicad_pcb (KiCad board)
At the start: 2 copper layers, 0 parts

Commit message: New: board outline and first raw component placement
Parts:
- added A1: 2500AT44M0400, Tom:2500AT44M0400, F.Cu at (196.5, 114.5)
- added C1: 18pF, SMD_Packages:SM0603_Capa, F.Cu at (130.5, 117.4)
- added C10: 10pF, SMD_Packages:SM0603_Capa, F.Cu at (194.5, 102.5)
- added C11: 1uF, SMD_Packages:SM0603_Capa, F.Cu at (174.0, 118.0)
- added C12: 1uF, SMD_Packages:SM0603_Capa, F.Cu at (181.0, 118.0)
- added C13: 10nF, SMD_Packages:SM0603_Capa, B.Cu at (145.7, 115.3)
- added C14: 10nF, SMD_Packages:SM0603_Capa, F.Cu at (158.1, 101.6)
- added C15: 0.1uF, SMD_Packages:SM0603_Capa, F.Cu at (156.4, 101.6)
- added C16: 2.2nF, SMD_Packages:SM0603_Capa, F.Cu at (155.6, 110.0)
- added C17: 0.1uF, SMD_Packages:SM0603_Capa, F.Cu at (161.4, 106.7)
- added C18: 100nF, SMD_Packages:SM0603_Capa, F.Cu at (157.6, 118.9)
- added C2: 18pF, SMD_Packages:SM0603_Capa, F.Cu at (136.6, 117.4)
- added C3: 100nF, SMD_Packages:SM0603_Capa, F.Cu at (126.9, 112.8)
- added C4: 100nF, SMD_Packages:SM0603_Capa, F.Cu at (149.0, 106.2)
- added C5: 220uF, 6.3V, Capacitors_SMD:c_elec_8x6.7, B.Cu at (132.0, 110.0)
- added C6: 220uF, 6.3V, Capacitors_SMD:c_elec_8x6.7, B.Cu at (107.0, 110.0)
- added C7: 470pF, SMD_Packages:SM0603_Capa, F.Cu at (107.3, 102.9)
- added C8: 220uF, 6.3V, Capacitors_SMD:c_elec_8x6.7, B.Cu at (157.5, 110.0)
- added C9: 2.2pF, SMD_Packages:SM0603_Capa, F.Cu at (196.5, 107.0)
- added D1: LED, LEDs:LED-0603, F.Cu at (140.9, 107.7)
- added K1: CONN_3, Socket_Strips:Socket_Strip_Straight_1x03, F.Cu at (116.5, 106.0)
- added K2: CONN_3, Socket_Strips:Socket_Strip_Straight_1x03, F.Cu at (116.5, 109.5)
- added K3: CONN_3, Socket_Strips:Socket_Strip_Straight_1x03, F.Cu at (116.5, 113.0)
- added L1: NC, SMD_Packages:SM0603, F.Cu at (194.5, 109.0)
- added L2: 2.2nH, SMD_Packages:SM0603, F.Cu at (194.5, 105.0)
- added MH: MountingHole_2-5mm_RevA_Date21Jun2010, Mounting_Holes:MountingHole_2-5mm, F.Cu at (167.5, 110.0)
- added MH: MountingHole_2-5mm_RevA_Date21Jun2010, Mounting_Holes:MountingHole_2-5mm, F.Cu at (124.0, 110.0)
- added P1: TST, Measurement_Points:Measurement_Point_Round-TH_Small, F.Cu at (132.2, 121.9)
- added P10: CONN_1, Socket_Strips:Socket_Strip_Straight_1x01, F.Cu at (124.0, 102.5)
- added P11: TST, Measurement_Points:Measurement_Point_Round-TH_Small, F.Cu at (177.7, 98.1)
- added P12: TST, Measurement_Points:Measurement_Point_Round-TH_Small, F.Cu at (180.0, 98.1)
- added P13: TST, Measurement_Points:Measurement_Point_Round-TH_Small, F.Cu at (182.3, 98.1)
- added P14: TST, Measurement_Points:Measurement_Point_Round-TH_Small, F.Cu at (184.6, 98.1)
- added P15: TST, Measurement_Points:Measurement_Point_Round-TH_Small, F.Cu at (181.0, 121.9)
- added P2: TST, Measurement_Points:Measurement_Point_Round-TH_Small, F.Cu at (142.7, 121.9)
- added P3: SWD_CONN, Tom:SWD_CONN, F.Cu at (145.2, 115.8)
- added P4: CONN_4, Socket_Strips:Socket_Strip_Straight_1x04, F.Cu at (101.0, 110.0)
- added P5: TST, Measurement_Points:Measurement_Point_Round-TH_Small, F.Cu at (135.0, 121.9)
- added P6: TST, Measurement_Points:Measurement_Point_Round-TH_Small, F.Cu at (155.1, 121.9)
- added P7: TST, Measurement_Points:Measurement_Point_Round-TH_Small, F.Cu at (137.3, 121.9)
- added P8: TST, Measurement_Points:Measurement_Point_Round-TH_Small, F.Cu at (152.6, 121.9)
- added P9: CONN_1, Socket_Strips:Socket_Strip_Straight_1x01, F.Cu at (124.0, 117.0)
- added R1: 10k, SMD_Packages:SM0603_Resistor, F.Cu at (131.5, 102.4)
- added R10: NC, SMD_Packages:SM0603_Resistor, F.Cu at (187.5, 101.5)
- added R12: 10k, SMD_Packages:SM0603_Resistor, B.Cu at (152.0, 103.7)
- added R13: 10k, SMD_Packages:SM0603_Resistor, B.Cu at (149.8, 103.7)
- added R14: 10k, SMD_Packages:SM0603_Resistor, B.Cu at (147.0, 103.7)
- added R15: 10k, SMD_Packages:SM0603_Resistor, B.Cu at (144.4, 103.7)
- added R16: 10k, SMD_Packages:SM0603_Resistor, B.Cu at (141.9, 103.7)
- added R17: 10k, SMD_Packages:SM0603_Resistor, B.Cu at (139.3, 103.7)
- added R18: 10k, SMD_Packages:SM0603_Resistor, B.Cu at (136.8, 103.7)
- added R2: 10k, SMD_Packages:SM0603_Resistor, F.Cu at (133.5, 102.4)
- added R3: 10k, SMD_Packages:SM0603_Resistor, F.Cu at (140.9, 117.1)
- added R4: 1.5k, SMD_Packages:SM0603_Resistor, F.Cu at (105.1, 111.3)
- added R5: 10k, SMD_Packages:SM0603_Resistor, F.Cu at (153.1, 114.3)
- added R6: 10k, SMD_Packages:SM0603_Resistor, F.Cu at (153.1, 112.5)
- added R7: 2k, SMD_Packages:SM0603_Resistor, F.Cu at (141.6, 110.3)
- added R8: 2k, SMD_Packages:SM0603_Resistor, F.Cu at (107.6, 118.9)
- added R9: OR, SMD_Packages:SM0603_Resistor, F.Cu at (180.0, 101.5)
- added U1: LPC11U3x, Tom:LQFP-48, F.Cu at (133.5, 110.0)
- added U2: M25P40, Tom:SO8N, F.Cu at (145.2, 106.2)
- added U3: TC1015-3.3, Tom:SOT-23-5, F.Cu at (107.5, 106.0)
- added U4: MCP73832, Tom:SOT-23-5, F.Cu at (107.5, 116.0)
- added U5: CC3000, Tom:CC3000, F.Cu at (180.5, 110.0)
- added U6: AT42QT1070, SOIC_Packages:SOIC-14_Narrow, B.Cu at (144.9, 110.0)
- added U7: MPU9150, Tom:LGA, F.Cu at (157.4, 105.9)
- added U8: MS5607, Tom:MS5607 Package, F.Cu at (157.6, 115.6)
- added X1: 12.000 MHz, Tom:CRYSTAL_SMD_3225, F.Cu at (133.5, 117.4)
- added capacitive1: CONN_7, Socket_Strips:Socket_Strip_Straight_1x07, F.Cu at (144.4, 99.6)
Other:
- board outline added: 100 x 21 mm

Commit message: New: Setup design rules and trace widths
Other:
- net class Default: clearance 0.254 -> 0.2; trace_width 0.254 -> 0.2; via_dia 0.889 -> 0.8; via_drill 0.635 -> 0.4
- rule trace_clearance: 0.254 -> 0.2
- rule trace_min: 0.254 -> 0.1524
- rule via_min_drill: 0.508 -> 0.3302
- rule via_min_size: 0.889 -> 0.6858
Changed lines of the file:
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@@
     (links 188)
     (no_connects 188)
-    (area 98.924999 99.424999 199.075001 120.575001)
+    (area 96.979115 93.798 202.917858 125.8972)
     (thickness 1.6)
     (drawings 20)
@@
   )
   (setup
-    (last_trace_width 0.254)
-    (trace_clearance 0.254)
+    (last_trace_width 0.8)
+    (user_trace_width 0.25)
+    (user_trace_width 0.4)
+    (user_trace_width 0.8)
+    (user_trace_width 1.5)
+    (trace_clearance 0.2)
     (zone_clearance 0.508)
     (zone_45_only no)
-    (trace_min 0.254)
+    (trace_min 0.1524)
     (segment_width 0.2)
     (edge_width 0.15)
-    (via_size 0.889)
-    (via_drill 0.635)
-    (via_min_size 0.889)
-    (via_min_drill 0.508)
+    (via_size 0.8)
+    (via_drill 0.4)
+    (via_min_size 0.6858)
+    (via_min_drill 0.3302)
     (uvia_size 0.508)
     (uvia_drill 0.127)
@@
   (net 66 "Net-(U5-Pad28)")
   (net_class Default "This is the default net class."
-    (clearance 0.254)
-    (trace_width 0.254)
-    (via_dia 0.889)
-    (via_drill 0.635)
+    (clearance 0.2)
+    (trace_width 0.2)
+    (via_dia 0.8)
+    (via_drill 0.4)
     (uvia_dia 0.508)
     (uvia_drill 0.127)
@@
     (add_net "Net-(P14-Pad1)")
     (add_net "Net-(P15-Pad1)")
-    (add_net "Net-(P3-Pad8)")
     (add_net "Net-(R12-Pad1)")
     (add_net "Net-(R12-Pad2)")
@@
     (add_net "Net-(R18-Pad2)")
     (add_net "Net-(R8-Pad1)")
-    (add_net "Net-(U1-Pad35)")
     (add_net "Net-(U5-Pad28)")
-    (add_net "Net-(U7-Pad5)")
     (add_net VBAT)
   )
